File: hw/eggbot.kicad_pcb (KiCad board)
At the start: 2 copper layers, 24 parts, among them J1 JACK_2P, K1 CONN_3, P1 CONN_2, P2 CONN_2, P3 CONN_4, P4 CONN_4, U1 ARDUINO_MINI_PRO, U2 7805, U3 POLOLU_STEPPER_CARRIER, U4 POLOLU_STEPPER_CARRIER

Commit message: Latest revision of schematics
Other:
- board outline added: 63.5 x 68.6 mm
Changed lines of the file:
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@@
     (links 59)
     (no_connects 0)
-    (area 44.45 25.273 132.46 106.84)
+    (area 44.399999 23.550879 132.46 106.84)
     (thickness 1.6)
-    (drawings 4)
+    (drawings 8)
     (tracks 178)
     (zones 0)
@@
     (pad_drill 2.99974)
     (pad_to_mask_clearance 0)
-    (aux_axis_origin 0 0)
+    (aux_axis_origin 44.45 25.4)
     (visible_elements FFFFFFBF)
     (pcbplotparams
-      (layerselection 3178497)
+      (layerselection 268435457)
       (usegerberextensions true)
       (excludeedgelayer true)
@@
       (viasonmask false)
       (mode 1)
-      (useauxorigin false)
+      (useauxorigin true)
       (hpglpennumber 1)
       (hpglpenspeed 20)
@@
       (outputformat 1)
       (mirror false)
-      (drillshape 1)
+      (drillshape 0)
       (scaleselection 1)
-      (outputdirectory ""))
+      (outputdirectory out/))
   )
   (net 0 "")
@@
     )
   )
+  (gr_line (start 107.95 25.4) (end 44.45 25.4) (angle 90) (layer Edge.Cuts) (width 0.1))
+  (gr_line (start 107.95 93.98) (end 107.95 25.4) (angle 90) (layer Edge.Cuts) (width 0.1))
+  (gr_line (start 44.45 93.98) (end 107.95 93.98) (angle 90) (layer Edge.Cuts) (width 0.1))
+  (gr_line (start 44.45 25.4) (end 44.45 93.98) (angle 90) (layer Edge.Cuts) (width 0.1))
   (gr_text "Egg v1" (at 97.79 35.56 315) (layer B.Cu)
     (effects (font (size 4 4) (thickness 0.9)) (justify mirror))
